File: Eagle/Frequency.brd (EAGLE design)
At the start: 213.4 x 49.5 mm, 24 parts

Commit message: More changes
Parts:
- moved E$24 15.2 mm to (167.6, 3.81)
- moved E$23 11.5 mm to (193.0, 3.81)
- moved E$22 11.4 mm to (193.0, 38.1)
- moved E$10 8.89 mm to (141.0, 26.7)
- moved E$17 8.89 mm to (148.6, 22.9)
- moved E$3 8.89 mm to (148.6, 33.0)
- moved E$19 7.62 mm to (104.1, 5.08)
- moved E$11 6.35 mm to (171.4, 26.7)
- moved E$18 6.35 mm to (179.1, 22.9)
- moved E$6 6.35 mm to (179.1, 33.0)
- moved E$12 5.08 mm to (110.5, 26.7)
- moved E$16 5.08 mm to (118.1, 22.9)
- moved E$2 5.08 mm to (118.1, 33.0)
- moved E$15 2.54 mm to (87.6, 22.9)
- moved E$4 2.54 mm to (87.6, 33.0)
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Other:
- board size 213.4 x 49.5 mm -> 200.7 x 49.5 mm
- board text added: "Frequency - V1.0"
