File: Eagle/Frequency.brd (EAGLE design)
At the start: 200.7 x 49.5 mm, 24 parts

Commit message: More changes
Parts:
- C1, C2, C3, C4, C5, C6: value (none) -> 100nf
- D1, D2, D3, D4, D5, D6: value (none) -> WS2812D
- R1, R2, R3, R4, R5, R6: value (none) -> 75
- renumbered E$1 to D2, E$10 to R5, E$11 to R6, E$12 to R4, E$13 to C1, E$14 to C2, E$15 to C3, E$16 to C4, E$17 to C5, E$18 to C6, E$19 to SW1, E$2 to D4, E$24 to CON1, E$3 to D5, E$4 to D3, E$5 to D1, E$6 to D6, E$7 to R1, E$8 to R2, E$9 to R3
Connections:
- new net S$1: C1.1, C2.1, C3.1, C4.1, C5.1, C6.1, CON1.5, D1.GND, D2.GND, D3.GND, D4.GND, D5.GND, D6.GND, SW1.2
- new net S$10: D6.DI, R6.2
- new net S$11: D5.DO, R6.1
- new net S$12: D4.DO, R5.1
- new net S$13: D3.DO, R4.1
- new net S$14: D2.DO, R3.1
- new net S$15: D1.DO, R2.1
- new net S$16: CON1.2, D6.DO
- new net S$2: C1.2, C2.2, C3.2, C4.2, C5.2, C6.2, CON1.4, D1.VCC, D2.VCC, D3.VCC, D4.VCC, D5.VCC, D6.VCC
- new net S$3: CON1.1, SW1.1
- new net S$4: CON1.3, R1.1
- new net S$5: D1.DI, R1.2
- new net S$6: D2.DI, R2.2
- new net S$7: D3.DI, R3.2
- new net S$8: D4.DI, R4.2
- new net S$9: D5.DI, R5.2
Other:
- board text added: "5 - GND 2 - DOUT 4 - 5v 1 - MODE 3 - DIN"
- board text removed: "5 - xxxxxxxxxx 2 - xxxxxxxxxx 4 - xxxxxxxxxx 1 - xxxxxxxxxx 3 - xxxxxxxxxx"

Commit message: More changes
Parts:
- moved CON1 2.54 mm to (170.2, 3.81)
- moved D1 1.02 mm to (26.7, 32.0)
- moved D2 1.02 mm to (57.1, 32.0)
- moved D3 1.02 mm to (87.6, 32.0)
- moved D4 1.02 mm to (118.1, 32.0)
- moved D5 1.02 mm to (148.6, 32.0)
- moved D6 1.02 mm to (179.1, 32.0)
Other:
- board text added: "5 - GND 2 - DOUT 4 - 5V 1 - MODE 3 - DIN"
- board text removed: "5 - GND 2 - DOUT 4 - 5v 1 - MODE 3 - DIN"
