File: Eagle/ESP32 30Pin Large Map.brd (EAGLE design)
At the start: 92.7 x 67.3 mm, 10 parts

Commit message: More changes
Routing:
- net S$2: track 0.00 -> 76.9 mm
- net S$1: track 0.00 -> 74.1 mm
- net S$3: track 0.00 -> 72.6 mm
- net S$5: track 0.00 -> 62.0 mm
- net S$6: track 0.00 -> 57.9 mm
- net S$4: track 0.00 -> 38.0 mm
Changed lines of the file:
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@@
 Large
 V1.0</text>
-<text x="16.51" y="3.81" size="1.778" layer="25">M.D.Waller G0PJO (c) Copyright 2024. All rights reserved.</text>
+<text x="15.24" y="3.81" size="1.6764" layer="25">M.D.Waller G0PJO (c) Copyright 2024. All rights reserved.</text>
 <text x="74.93" y="26.67" size="1.016" layer="25" rot="R90">5V</text>
 <text x="74.93" y="21.59" size="1.016" layer="25" rot="R90">GND</text>
@@
 <contactref element="LEDS" pad="1"/>
 <contactref element="U1" pad="VIN"/>
-<wire x1="16.51" y1="20.32" x2="83.82" y2="27.8638" width="0" layer="19" extent="1-1"/>
+<wire x1="40.2336" y1="20.2692" x2="16.6116" y2="20.2692" width="0.1524" layer="1"/>
+<wire x1="44.5008" y1="16.002" x2="40.2336" y2="20.2692" width="0.1524" layer="1"/>
+<wire x1="72.0852" y1="16.002" x2="44.5008" y2="16.002" width="0.1524" layer="1"/>
+<wire x1="83.82" y1="27.7368" x2="72.0852" y2="16.002" width="0.1524" layer="1"/>
+<wire x1="16.6116" y1="20.2692" x2="16.51" y2="20.32" width="0.1524" layer="1"/>
+<wire x1="83.82" y1="27.7368" x2="83.82" y2="27.8638" width="0.1524" layer="1"/>
 </signal>
 <signal name="S$2">
 <contactref element="U1" pad="GND"/>
 <contactref element="LEDS" pad="2"/>
-<wire x1="16.51" y1="22.86" x2="83.82" y2="22.86" width="0" layer="19" extent="1-1"/>
+<wire x1="16.4592" y1="22.098" x2="16.4592" y2="22.86" width="0.1524" layer="1"/>
+<wire x1="15.24" y1="20.8788" x2="16.4592" y2="22.098" width="0.1524" layer="1"/>
+<wire x1="15.24" y1="19.812" x2="15.24" y2="20.8788" width="0.1524" layer="1"/>
+<wire x1="19.3548" y1="15.6972" x2="15.24" y2="19.812" width="0.1524" layer="1"/>
+<wire x1="76.6572" y1="15.6972" x2="19.3548" y2="15.6972" width="0.1524" layer="1"/>
+<wire x1="83.82" y1="22.86" x2="76.6572" y2="15.6972" width="0.1524" layer="1"/>
+<wire x1="16.4592" y1="22.86" x2="16.51" y2="22.86" width="0.1524" layer="1"/>
 </signal>
 <signal name="S$3">
 <contactref element="LEDS" pad="3"/>
 <contactref element="U1" pad="D14"/>
-<wire x1="16.51" y1="30.48" x2="83.82" y2="17.8562" width="0" layer="19" extent="1-1"/>
+<wire x1="30.0228" y1="30.48" x2="16.51" y2="30.48" width="0.1524" layer="16"/>
+<wire x1="42.2148" y1="18.288" x2="30.0228" y2="30.48" width="0.1524" layer="16"/>
+<wire x1="83.5152" y1="18.288" x2="42.2148" y2="18.288" width="0.1524" layer="16"/>
+<wire x1="83.82" y1="17.9832" x2="83.5152" y2="18.288" width="0.1524" layer="16"/>
+<wire x1="83.82" y1="17.9832" x2="83.82" y2="17.8562" width="0.1524" layer="16"/>
 </signal>
 <signal name="S$4">
 <contactref element="R1" pad="1"/>
 <contactref element="U1" pad="D25"/>
-<wire x1="16.51" y1="38.1" x2="50.8" y2="46.99" width="0" layer="19" extent="1-1"/>
+<wire x1="25.4508" y1="46.9392" x2="50.7492" y2="46.9392" width="0.1524" layer="1"/>
+<wire x1="16.6116" y1="38.1" x2="25.4508" y2="46.9392" width="0.1524" layer="1"/>
+<wire x1="50.7492" y1="46.9392" x2="50.8" y2="46.99" width="0.1524" layer="1"/>
+<wire x1="16.6116" y1="38.1" x2="16.51" y2="38.1" width="0.1524" layer="1"/>
 </signal>
 <signal name="S$5">
@@
 <contactref element="U1" pad="GND@1"/>
 <contactref element="MODE" pad="2"/>
-<wire x1="50.8" y1="33.02" x2="83.82" y2="36.8554" width="0" layer="19" extent="1-1"/>
-<wire x1="41.91" y1="22.86" x2="50.8" y2="33.02" width="0" layer="19" extent="1-1"/>
-<wire x1="61.94" y1="17.22" x2="50.8" y2="33.02" width="0" layer="19" extent="1-1"/>
+<wire x1="50.7492" y1="31.6992" x2="50.7492" y2="32.9184" width="0.1524" layer="1"/>
+<wire x1="41.91" y1="22.86" x2="49.53" y2="30.48" width="0.1524" layer="1"/>
+<wire x1="49.53" y1="30.48" x2="50.7492" y2="31.6992" width="0.1524" layer="1"/>
+<wire x1="50.7492" y1="32.9184" x2="50.8" y2="33.02" width="0.1524" layer="1"/>
+<wire x1="61.8744" y1="18.1356" x2="61.8744" y2="17.2212" width="0.1524" layer="1"/>
+<wire x1="49.53" y1="30.48" x2="61.8744" y2="18.1356" width="0.1524" layer="1"/>
+<wire x1="61.8744" y1="17.2212" x2="61.94" y2="17.22" width="0.1524" layer="1"/>
+<wire x1="80.4672" y1="36.7284" x2="83.82" y2="36.7284" width="0.1524" layer="1"/>
+<wire x1="61.8744" y1="18.1356" x2="80.4672" y2="36.7284" width="0.1524" layer="1"/>
+<wire x1="83.82" y1="36.7284" x2="83.82" y2="36.8554" width="0.1524" layer="1"/>
 </signal>
 <signal name="S$6">
@@
 <contactref element="R1" pad="2"/>
 <contactref element="MODE" pad="1"/>
-<wire x1="50.8" y1="27.94" x2="83.82" y2="41.8846" width="0" layer="19" extent="1-1"/>
-<wire x1="50.8" y1="36.83" x2="50.8" y2="27.94" width="0" layer="19" extent="1-1"/>
-<wire x1="57.44" y1="17.22" x2="50.8" y2="27.94" width="0" layer="19" extent="1-1"/>
+<wire x1="50.9016" y1="31.8516" x2="50.9016" y2="28.0416" width="0.1524" layer="16"/>
+<wire x1="51.816" y1="32.766" x2="50.9016" y2="31.8516" width="0.1524" layer="16"/>
+<wire x1="51.816" y1="35.814" x2="51.816" y2="32.766" width="0.1524" layer="16"/>
+<wire x1="50.8" y1="36.83" x2="51.816" y2="35.814" width="0.1524" layer="16"/>
+<wire x1="50.9016" y1="28.0416" x2="50.8" y2="27.94" width="0.1524" layer="16"/>
+<wire x1="57.3024" y1="21.4884" x2="57.3024" y2="17.2212" width="0.1524" layer="1"/>
+<wire x1="50.9016" y1="27.8892" x2="57.3024" y2="21.4884" width="0.1524" layer="1"/>
+<wire x1="57.3024" y1="17.2212" x2="57.44" y2="17.22" width="0.1524" layer="1"/>
+<wire x1="50.9016" y1="27.8892" x2="50.8" y2="27.94" width="0.1524" layer="1"/>
+<wire x1="57.7596" y1="41.7576" x2="83.82" y2="41.7576" width="0.1524" layer="16"/>
+<wire x1="51.816" y1="35.814" x2="57.7596" y2="41.7576" width="0.1524" layer="16"/>
+<wire x1="83.82" y1="41.7576" x2="83.82" y2="41.8846" width="0.1524" layer="16"/>
 </signal>
 </signals>
